File: z-axis-addon.kicad_sch (KiCad schematic)
At the start: 9 parts, among them J1 Conn_01x06_Socket, J2 Conn_01x08_Socket, J3 Conn_01x03_Socket, J4 Conn_01x04_Socket, U1 TMC2130

Commit message: Update schematic to include power led
Parts:
- D1: footprint (none) -> LED_SMD:LED_0805_2012Metric
- R2: footprint (none) -> Resistor_SMD:R_0805_2012Metric
Changed lines of the file:
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@@
 			)
 		)
-		(property "Footprint" ""
+		(property "Footprint" "LED_SMD:LED_0805_2012Metric"
 			(at 63.5 74.93 0)
 			(effects
@@
 			)
 		)
-		(property "Footprint" ""
+		(property "Footprint" "Resistor_SMD:R_0805_2012Metric"
 			(at 61.722 63.5 90)
 			(effects
